File: Hardware/Adj.sch (EAGLE design)
At the start: 53 parts, among them Q1 BSS84, Q2 2N7002, Q3 Si2307, U1 LM317, U2 NOKIA5110ALT-TOP, U3 LM358, U4 MEGA8-P, U6 LD117AS33TR, U7 ICL7660CPA

Commit message: update 1
Parts:
- added L1: 600R, ipc-7351-resistor:RESISTOR_0603
Connections:
- new net N$1: C5.2, L1.2, U4.AVCC
- net +3.3V: now also L1.1; no longer C5.2, U4.AVCC
Other:
- note added: "Ferrite"
- moved on the sheet: C2, C20, C3, C5, C8, R13, R15, U6

Commit message: clean u 1
Parts:
- added D5: 1N4148, diode:1N4148DO35-7
- C1, C14, C15, C16, C17, C18, C19, C2, C3, C4, C5, C6, D2, D3, D4, Q1, Q2, Q3, R1, R10, R11, R12, R13, R14, R15, R16, R17, R18, R2, R3, R4, R6, R7, R8, R9, U1, U3, U6: PARTNO (none) -> *
- C10: PARTNO (none) -> 47uF/25V
- C11, C12, C8: PARTNO (none) -> 10uF/25V
- C13: value 10uF -> 47uF; PARTNO (none) -> 47uF/25V
- C20, C7, C9: PARTNO (none) -> 100uF/25V
- D1: value (none) -> 1N4148; device ipc-7351-diode:KA2KA_SOT-23 -> diode:1N4148DO35-7; PARTNO (none) -> *
- JP1: value (none) -> 2x3 header; PARTNO (none) -> *
- JP2: value (none) -> Rotary enoder; PARTNO (none) -> *
- L1: PARTNO (none) -> Ferrite 600R@100MHz
- R5: PARTNO (none) -> 0R1 1W
- U2: value NOKIA5110ALT-TOP -> NOKIA5110; PARTNO (none) -> Nokia 5110 LCD
- U4: PARTNO (none) -> ATMerga8A
- U7: PARTNO (none) -> ICL7660CPA
Connections:
- net N$14: now also D1.C, D5.A; no longer D1.KA
- net VDD: now also D5.C; no longer D1.K
Other:
- note added: "10uF: 10uF/25V Electrolytic 47uF: 47uF/25V Electrolytic 100uF: 100uF/25V Electrolytic"
- note removed: "10uF: 10uF/25V Electrolytic 100uF: 100uF/25V Electrolytic"
- moved on the sheet: C13
